Commit message: urdf examples

File: roboticstoolbox/robot/robot.urdf (robot description, URDF)
Before this commit: robot robotRTB, 10 links, 9 joints
Links:
- removed link link5
- removed link link6
- removed link link7
Joints:
- removed joint joint5
- removed joint joint6
- removed joint joint7
- joint ee_joint: origin xyz=0.0 0.0 0.10300000000000001 rpy=0.0 -0.0 -0.7853981633974483 -> xyz=0.05547001962252285 -0.08320502943378433 0.0 rpy=0.0 -0.0 -0.9827937232473289; parent link7 -> link4
- joint joint1: origin xyz=0.0 0.0 0.333 rpy=0.0 -0.0 0.0 -> xyz=0.0 0.0 0.0 rpy=0.0 -0.0 0.0
- joint joint2: origin xyz=0.0 0.0 0.0 rpy=-1.5707963267948966 -0.0 0.0 -> xyz=0.0 0.0 0.2 rpy=0.0 -1.5707963267948966 -1.5707963267948966
- joint joint3: limit (none) -> lower=0.0 upper=1.0 effort=10 velocity=1.0; origin xyz=0.0 -0.316 1.934941942652818e-17 rpy=1.5707963267948966 -0.0 0.0 -> xyz=0.0 0.0 0.0 rpy=0.0 -0.0 0.0; type continuous -> prismatic
- joint joint4: origin xyz=0.0825 0.0 0.0 rpy=1.5707963267948966 -0.0 0.0 -> xyz=0.3 0.2 0.0 rpy=3.141592653589793 -0.0 0.5880026035475676
